File: advancedRGBmod/Main-PCB/n64adv2.sch (EAGLE design)
At the start: 158 parts, among them U1 10CL025YE144, U2 ADV7513, U3 S25FLXXXSO8-DUAL, U4 27M, U5 TLV70212DBVT, U6 TLV70225DBVT, U7 TLV70218DBVT, U8 TLV70033, X1 FH12-24S-0.5SH, X3 hdmi-con, X4 2510-

Commit message: remove connections for DE and MCLK and change pinout for system LEDs
Parts:
- removed R25: 50, rcl:R-EU_R0603
Connections:
- removed net N$26: U1.IO85, U2.DE
- removed net N$29: RN15.4, U2.MCLK
- removed net N$56: RN15.8, U1.IO72/PLL4_CLKON
- new net N$15: D1.C, U1.IO72/PLL4_CLKON
- net GND: now also U2.DE, U2.MCLK; no longer R25.2
- net N$11: now also U1.VREF/IO80; no longer U1.IO71/PLL4_CLKOP
- net N$13: now also U1.IO71/PLL4_CLKOP; no longer U1.IO49
- net N$27: now also U1.IO85; no longer U1.IO83
- net N$28: now also U1.IO83; no longer U1.VREF/IO80
- net N$30: now also RN15.4; no longer RN15.3
- net N$31: now also RN15.3; no longer RN15.2
- net N$32: now also RN15.2; no longer RN15.1
- net N$62: no longer D1.C
- net TX_CLK: no longer R25.1
Other:
- note added: "Schematic (c) 2018 by Peter Bartmann aka borti4938 Version: N64Av2_20181111"
- note removed: "Schematic (c) 2018 by Peter Bartmann aka borti4938"
- moved on the sheet: D1, D2, DR1, DR2, R17
